File: hardware/raspi-rfid-rc522.brd (EAGLE design)
At the start: 67.3 x 36.8 mm, 7 parts

Commit message: update pcb
Parts:
- removed JP2: NEOPIXEL RING, pinhead:1X03
- removed JP3: Battery Pack, pinhead:1X03
- added 2124: B G 5V, pinhead:1X03
- added A_I2C: A_SDA A_SCL, pinhead:1X02
- added NEOPIXEL: (no value), pinhead:1X03
- added P_I2C: (no value), pinhead:1X02
- moved R2 2.90 mm to (37.0, 6.10), turned to 0 degrees
- moved R1 1.08 mm to (40.8, 9.65), turned to 180 degrees
- turned U$1 to 0 degrees
Connections:
- new net A_RST: U$1.RST, U$2.29
- new net A_SCL: A_I2C.2, U$1.SCL
- new net A_SDA: A_I2C.1, U$1.SDA
- new net GPIO13: U$1.13, U$2.33
- new net IRQ: JP1.4, U$2.18
- net 2: now also NEOPIXEL.1; no longer JP2.1
- net 3V3: now also NEOPIXEL.2; no longer JP2.2
- net 5V: now also 2124.3; no longer JP3.3
- net BAT: now also 2124.1; no longer JP3.1
- net GND: now also 2124.2, NEOPIXEL.3; no longer JP2.3, JP3.2
- net SCL: now also P_I2C.2
- net SDA: now also P_I2C.1
Routing:
- net 2: track 62.6 -> 4.45 mm
- net BAT: track 25.6 -> 70.5 mm, vias 2 -> 1
- net A_RST: track 0.00 -> 33.9 mm
- net SCL: track 15.1 -> 44.9 mm, vias 0 -> 1
- net 5V: track 46.0 -> 73.6 mm, vias 1 -> 0
- net SDA: track 19.0 -> 46.4 mm, vias 0 -> 1
- net IRQ: track 0.00 -> 17.6 mm
- net GPIO12: track 23.0 -> 9.42 mm
- net GPIO13: track 0.00 -> 11.9 mm
- net A_SDA: track 0.00 -> 9.27 mm
- net A_SCL: track 0.00 -> 9.27 mm
- net RST: track 31.0 -> 27.5 mm
Other:
- board text added: "(c) Jared Mauch"
- board text added: "SCL"
- board text added: "SDA"
