File: hardware/raspi-rfid-rc522.sch (EAGLE design)
At the start: 7 parts

Commit message: update pcb
Parts:
- removed JP3: Battery Pack, pinhead:PINHD-1X3
- added 2124: B G 5V, pinhead:PINHD-1X3
- added A_I2C: A_SDA A_SCL, pinhead:PINHD-1X2
- added P_I2C: (no value), pinhead:PINHD-1X2
- NEOPIXEL: value NEOPIXEL RING -> (none)
- renumbered JP2 to NEOPIXEL
Connections:
- new net A_RST: U$1.RST, U$2.GPIO5
- new net A_SCL: A_I2C.2, U$1.SCL
- new net A_SDA: A_I2C.1, U$1.SDA
- new net GPIO13: U$1.13, U$2.GPIO13
- new net IRQ: JP1.4, U$2.GEN5/GPIO24
- net 5V: now also 2124.3; no longer JP3.3
- net BAT: now also 2124.1; no longer JP3.1
- net GND: now also 2124.2; no longer JP3.2
- net SCL: now also P_I2C.2
- net SDA: now also P_I2C.1
Other:
- moved on the sheet: U$2
